Commit message: Update home position and author in README

File: src/ros2_kortex/kortex_description/robots/gen3_lite.urdf (robot description, URDF)
Before this commit: robot gen3_lite, 15 links, 14 joints
Joints:
- joint left_finger_tip_joint: mimic joint=right_finger_bottom_joint multiplier=-0.276 offset=0.0 -> joint=right_finger_bottom_joint multiplier=-0.676 offset=0.149
- joint right_finger_tip_joint: mimic joint=right_finger_bottom_joint multiplier=-0.276 offset=0.0 -> joint=right_finger_bottom_joint multiplier=-0.676 offset=0.149
