Commit message: Complete pick-and-place demo with optimizations
- Updated object positions to match between SDF and Python script
- Increased velocity/acceleration scaling to 0.8 (80%) for faster execution
- Reduced motion duration to 1.0 seconds
- Removed RViz marker publishing (objects static in Gazebo)
- Fixed physics configuration (2ms step with 500 Hz update rate)
- Added MATLAB joint angle streaming capability
- Updated README with comprehensive documentation
- Corrected home position in FK script to match implementation
- Fixed gripper mimic joint limits in XACRO files

File: src/ros2_kortex/kortex_description/grippers/gen3_lite_2f/urdf/gen3_lite_2f_macro.xacro (robot description, xacro)
@@ -138,6 +138,5 @@
         <child link="${prefix}right_finger_dist_link" />
         <axis xyz="0 0 1" />
-        <limit lower="-1.03" upper="0.21" effort="1000" velocity="1000" />
-        <!--limit lower="-1.03" upper="0.21" effort="1000" velocity="1000" /-->
+        <limit lower="-0.50" upper="0.21" effort="1000" velocity="1000" /> <!--limit lower="-1.03" upper="0.21" effort="1000" velocity="1000" /-->
         <mimic joint="${prefix}right_finger_bottom_joint" multiplier="-0.276" offset="-0.1" />
       </joint>
@@ -206,6 +205,5 @@
         <child link="${prefix}left_finger_dist_link" />
         <axis xyz="0 0 -1" />
-        <limit lower="-1.03" upper="0.21" effort="1000" velocity="1000" />
-        <!--limit lower="-1.03" upper="0.21" effort="1000" velocity="1000" /-->
+        <limit lower="-0.50" upper="0.21" effort="1000" velocity="1000" /> <!--limit lower="-1.03" upper="0.21" effort="1000" velocity="1000" /-->
         <mimic joint="${prefix}right_finger_bottom_joint" multiplier="-0.276" offset="-0.1" />
       </joint>
@@ -317,6 +315,5 @@
         <child link="${prefix}right_finger_dist_link" />
         <axis xyz="0 0 1" />
-        <limit lower="-1.03" upper="0.21" effort="1000" velocity="1000" />
-        <!--limit lower="-1.03" upper="0.21" effort="1000" velocity="1000" /-->
+        <limit lower="-0.50" upper="0.21" effort="1000" velocity="1000" /> <!--limit lower="-1.03" upper="0.21" effort="1000" velocity="1000" /-->
         <mimic joint="${prefix}right_finger_bottom_joint" multiplier="-0.276" offset="-0.1" />
       </joint>
@@ -384,6 +381,5 @@
         <child link="${prefix}left_finger_dist_link" />
         <axis xyz="0 0 -1" />
-        <limit lower="-1.03" upper="0.21" effort="1000" velocity="1000" />
-        <!--limit lower="-1.03" upper="0.21" effort="1000" velocity="1000" /-->
+        <limit lower="-0.50" upper="0.21" effort="1000" velocity="1000" /> <!--limit lower="-1.03" upper="0.21" effort="1000" velocity="1000" /-->
         <mimic joint="${prefix}right_finger_bottom_joint" multiplier="-0.276" offset="-0.1" />
       </joint>
@@ -493,6 +489,5 @@
       <child link="right_finger_dist_link" />
       <axis xyz="0 0 1" />
-      <limit lower="-1.03" upper="0.21" effort="1000" velocity="1000" />
-       <!--limit lower="-1.03" upper="0.21" effort="1000" velocity="1000" /-->
+      <limit lower="-0.50" upper="0.21" effort="1000" velocity="1000" /> <!--limit lower="-1.03" upper="0.21" effort="1000" velocity="1000" /-->
       <mimic joint="right_finger_bottom_joint" multiplier="-0.676" offset="0.149" />
     </joint>
@@ -560,6 +555,5 @@
       <child link="left_finger_dist_link" />
       <axis xyz="0 0 -1" />
-      <limit lower="-1.03" upper="0.21" effort="1000" velocity="1000" />
-       <!--limit lower="-1.03" upper="0.21" effort="1000" velocity="1000" /-->
+      <limit lower="-0.50" upper="0.21" effort="1000" velocity="1000" /> <!--limit lower="-1.03" upper="0.21" effort="1000" velocity="1000" /-->
       <mimic joint="right_finger_bottom_joint" multiplier="-0.676" offset="0.149" />
     </joint>

Commit message: Update ros2_kortex workspace

File: src/ros2_kortex/kortex_description/grippers/gen3_lite_2f/urdf/gen3_lite_2f_macro.xacro (robot description, xacro)
@@ -138,6 +138,6 @@
         <child link="${prefix}right_finger_dist_link" />
         <axis xyz="0 0 1" />
-        <limit lower="-0.50" upper="0.21" effort="1000" velocity="1000" /> <!--limit lower="-1.03" upper="0.21" effort="1000" velocity="1000" /-->
-        <mimic joint="${prefix}right_finger_bottom_joint" multiplier="-0.276" offset="-0.1" />
+        <limit lower="-1.03" upper="0.21" effort="1000" velocity="1000" />
+        <mimic joint="${prefix}right_finger_bottom_joint" multiplier="-0.676" offset="0.149" />
       </joint>
       <link name="${prefix}left_finger_prox_link">
@@ -205,6 +205,6 @@
         <child link="${prefix}left_finger_dist_link" />
         <axis xyz="0 0 -1" />
-        <limit lower="-0.50" upper="0.21" effort="1000" velocity="1000" /> <!--limit lower="-1.03" upper="0.21" effort="1000" velocity="1000" /-->
-        <mimic joint="${prefix}right_finger_bottom_joint" multiplier="-0.276" offset="-0.1" />
+        <limit lower="-1.03" upper="0.21" effort="1000" velocity="1000" />
+        <mimic joint="${prefix}right_finger_bottom_joint" multiplier="-0.676" offset="0.149" />
       </joint>
     </xacro:unless>
